Commit message: problem with parsing

File: src/description/urdf/carlikebot_description.urdf.xacro (robot description, xacro)
@@ -1,40 +1,35 @@
 <?xml version="1.0"?>
-<robot xmlns:xacro="http://www.ros.org/wiki/xacro">
+<robot xmlns:xacro="http://www.ros.org/wiki/xacro" >
+  <!-- Macro definition for carlikebot -->
   <xacro:macro name="carlikebot" params="prefix">
-  <!-- Constants for robot dimensions -->
-  <xacro:property name="PI" value="3.1415926535897931"/>
-  <xacro:property name="base_mass" value="4.0" /> <!-- arbitrary value for base mass -->
-  <xacro:property name="base_width" value="0.260" />
-  <xacro:property name="base_length" value="0.525" />
-  <xacro:property name="base_height" value="0.060" />
-  <xacro:property name="wheelbase" value="0.325" />
-  <xacro:property name="wheel_mass" value="0.34055" /> <!-- arbitrary value for wheel mass -->
-  <xacro:property name="wheel_len" value="0.045" />
-  <xacro:property name="wheel_radius" value="0.05" />
-  <!-- <xacro:property name="wheeltrack" value="" -->
-  <!-- Base Link -->
-  <link name="${prefix}base_link" />
-  <!-- Chassis -->
-  <link name="${prefix}chassis_link">
-    <collision>
-      <origin xyz="0 0 0" rpy="0 0 0"/>
-      <geometry>
-        <box size="${base_length} ${base_width} ${base_height}"/>
-      </geometry>
-    </collision>
-    <visual>
-      <origin xyz="0 0 0" rpy="0 0 0"/>
-      <geometry>
-        <box size="${base_length} ${base_width} ${base_height}"/>
-      </geometry>
-      <material name="orange"/>
-    </visual>
-    <inertial>
-      <origin xyz="0 0 0" rpy="0 0 0"/>
-      <mass value="${base_mass}"/>
-        <inertia
-          ixx="0.000270" ixy="0.0" ixz="0.0"
-          iyy="0.000270" iyz="0.0"
-          izz="0.000426"/>
+    <!-- Constants for robot dimensions -->
+    <xacro:property name="PI" value="3.1415926535897931"/>
+    <xacro:property name="base_mass" value="4.0" />
+    <xacro:property name="base_width" value="0.408" />
+    <xacro:property name="base_length" value="0.558" />
+    <xacro:property name="base_height" value="0.060" />
+    <xacro:property name="wheelbase" value="0.558" />
+    <xacro:property name="wheel_mass" value="0.34055" />
+    <xacro:property name="wheel_len" value="0.05" />
+    <xacro:property name="wheel_radius" value="0.1" />
+    <!--Property	Value (m)	Description
+base_width	0.408	Track width (distance between wheels on the same axle).
+base_length	0.558	Total length of the robot base.
+wheelbase	0.558	Distance between the front and rear wheel axles.
+wheel_radius	0.1	Radius of each wheel (half the diameter).
+wheel_len	0.05	Width of the wheels.
+base_height	0.06	Height of the chassis.
+base_mass	Approximate weight of the chassis (adjust if known).-->
+    <!-- Base Link -->
+    <link name="${prefix}base_link" />
+    <!-- Chassis -->
+    <link name="${prefix}chassis_link">
+      <inertial>
+        <origin xyz="0 0 0" rpy="0 0 0"/>
+        <mass value="${base_mass}"/>
+        <inertia
+          ixx="0.001" ixy="0.0" ixz="0.0"
+          iyy="0.001" iyz="0.0"
+          izz="0.001"/>
       </inertial>
     </link>
@@ -42,49 +37,25 @@
       <parent link="${prefix}base_link"/>
       <child link="${prefix}chassis_link"/>
-      <origin xyz="0 0 ${base_height/2 + wheel_radius}" rpy="0 0 0"/>
+      <origin xyz="${wheelbase/2} 0 ${2*wheel_radius}" rpy="0 0 0"/>
+    </joint>
+    <!-- Rear Wheels -->
+    <!-- Virtual Rear Wheel -->
+    <link name="${prefix}virtual_rear_wheel" />
+    <joint name="${prefix}virtual_rear_wheel_joint" type="revolute">
+      <parent link="${prefix}chassis_link"/>
+      <child link="${prefix}virtual_rear_wheel"/>
+      <origin xyz="${wheelbase/2} 0 ${wheel_radius}" rpy="0 0 ${PI/2}"/>
       <axis xyz="0 0 1"/>
-      <dynamics damping="0.2"/>
-    </joint>
-    <!-- rear wheels -->
-    <!-- virtual rear wheel -->
-    <link name="${prefix}virtual_rear_wheel">
-      <visual>
-        <origin xyz="0 0 0" rpy="${PI/2} 0 ${PI/2}"/>
-        <geometry>
-          <cylinder length="0.01" radius="${wheel_radius}"/>
-        </geometry>
-        <material name="invisible"/>
-      </visual>
-    </link>
-    <joint name="${prefix}virtual_rear_wheel_joint" type="continuous">
-      <parent link="${prefix}chassis_link"/>
-      <child link="${prefix}virtual_rear_wheel"/>
-      <origin xyz="-${wheelbase/2} 0 -${base_height/2}" rpy="0 0 ${PI/2}"/>
-      <axis xyz="1 0 0"/>
-      <limit effort="100.0" velocity="100.0"/>
-      <dynamics damping="0.2"/>
-    </joint>
-    <!-- rear right wheel -->
+      <limit lower="-0.4" upper="0.4" effort="10.0" velocity="10.0"/>
+    </joint>
+    <!-- Rear Right Wheel -->
     <link name="${prefix}rear_right_wheel">
-      <collision>
-        <origin xyz="0 0 0" rpy="${PI/2} 0 ${PI/2}"/>
-        <geometry>
-          <cylinder length="${wheel_len}" radius="${wheel_radius}"/>
-        </geometry>
-      </collision>
-      <visual>
-        <origin xyz="0 0 0" rpy="${PI/2} 0 ${PI/2}"/>
-        <geometry>
-          <cylinder length="${wheel_len}" radius="${wheel_radius}"/>
-        </geometry>
-        <material name="black"/>
-      </visual>
-      <inertial>
-        <origin xyz="0 0 0" rpy="${PI/2} 0 ${PI/2}"/>
-        <mass value="${wheel_mass}"/>
-        <inertia
-          ixx="0.000270" ixy="0.0" ixz="0.0"
-          iyy="0.000270" iyz="0.0"
-          izz="0.000426"/>
+      <inertial>
+        <origin xyz="0 0 0" rpy="${PI/2} 0 ${PI/2}"/>
+        <mass value="${wheel_mass}"/>
+        <inertia
+          ixx="0.001" ixy="0.0" ixz="0.0"
+          iyy="0.001" iyz="0.0"
+          izz="0.001"/>
       </inertial>
     </link>
@@ -92,127 +63,140 @@
       <parent link="${prefix}chassis_link"/>
       <child link="${prefix}rear_right_wheel"/>
-      <origin xyz="-${wheelbase/2} ${base_width/2} -${base_height/2}" rpy="0 0 ${PI/2}"/>
-      <axis xyz="1 0 0"/>
-      <limit effort="100.0" velocity="100.0"/>
-      <dynamics damping="0.2"/>
+      <origin xyz="0 ${base_width/2} ${wheel_radius}" rpy="0 0 ${PI/2}"/>
+      <axis xyz="1 0 0"/>
+      <limit effort="10.0" velocity="10.0"/>
       <mimic joint="${prefix}virtual_rear_wheel_joint" multiplier="1.0" offset="0.0"/>
     </joint>
-    <!-- rear left wheel -->
+    <!-- Rear Left Wheel -->
     <link name="${prefix}rear_left_wheel">
-        <collision>
-          <origin xyz="0 0 0" rpy="${PI/2} 0 ${PI/2}"/>
-          <geometry>
-            <cylinder length="${wheel_len}" radius="${wheel_radius}"/>
-          </geometry>
-        </collision>
-        <visual>
-          <origin xyz="0 0 0" rpy="${PI/2} 0 ${PI/2}"/>
-          <geometry>
-            <cylinder length="${wheel_len}" radius="${wheel_radius}"/>
-          </geometry>
-          <material name="black"/>
-        </visual>
-        <inertial>
-          <origin xyz="0 0 0" rpy="${PI/2} 0 ${PI/2}"/>
-          <mass value="${wheel_mass}"/>
-          <inertia
-            ixx="0.000270" ixy="0.0" ixz="0.0"
-            iyy="0.000270" iyz="0.0"
-            izz="0.000426"/>
-        </inertial>
+      <inertial>
+        <origin xyz="0 0 0" rpy="${PI/2} 0 ${PI/2}"/>
+        <mass value="${wheel_mass}"/>
+        <inertia
+          ixx="0.001" ixy="0.0" ixz="0.0"
+          iyy="0.001" iyz="0.0"
+          izz="0.001"/>
+      </inertial>
     </link>
     <joint name="${prefix}rear_left_wheel_joint" type="continuous">
-      <parent link="${prefix}chassis_link" />
-      <child link="${prefix}rear_left_wheel" />
-      <origin xyz="-${wheelbase/2} -${base_width/2} -${base_height/2}" rpy="0 0 ${PI/2}"/>
-      <axis xyz="1 0 0"/>
-      <limit effort="100.0" velocity="100.0"/>
-      <dynamics damping="0.2"/>
+      <parent link="${prefix}chassis_link"/>
+      <child link="${prefix}rear_left_wheel"/>
+      <origin xyz="0 -${base_width/2} ${wheel_radius}" rpy="0 0 ${PI/2}"/>
+      <axis xyz="1 0 0"/>
+      <limit effort="10.0" velocity="10.0"/>
       <mimic joint="${prefix}virtual_rear_wheel_joint" multiplier="1.0" offset="0.0"/>
     </joint>
-    <!-- front wheels -->
-    <!-- virtual front wheel -->
-    <link name="${prefix}virtual_front_wheel">
-      <visual>
-        <origin xyz="0 0 0" rpy="${PI/2} 0 ${PI/2}"/>
-        <geometry>
-          <cylinder length="0.01" radius="${wheel_radius}"/>
-        </geometry>
-        <material name="invisible"/>
-      </visual>
-    </link>
+    <!-- Front Wheels -->
+    <!-- Virtual Front Wheel -->
+    <link name="${prefix}virtual_front_wheel" />
     <joint name="${prefix}virtual_front_wheel_joint" type="revolute">
       <parent link="${prefix}chassis_link"/>
       <child link="${prefix}virtual_front_wheel"/>
-      <origin xyz="${wheelbase/2} 0 -${base_height/2}" rpy="0 0 ${PI/2}"/>
+      <origin xyz="${wheelbase/2} 0 ${wheel_radius}" rpy="0 0 ${PI/2}"/>
       <axis xyz="0 0 1"/>
-      <limit lower="-0.4" upper="0.4" effort="100.0" velocity="0.0"/>
-      <dynamics damping="0.2"/>
-    </joint>
-    <!-- front right wheel -->
+      <limit lower="-0.4" upper="0.4" effort="10.0" velocity="10.0"/>
+    </joint>
+    <!-- Front Right Wheel -->
     <link name="${prefix}front_right_wheel">
-      <collision>
-        <origin xyz="0 0 0" rpy="${PI/2} 0 ${PI/2}"/>
-        <geometry>
-          <cylinder length="${wheel_len}" radius="${wheel_radius}"/>
-        </geometry>
-      </collision>
-      <visual>
-        <origin xyz="0 0 0" rpy="${PI/2} 0 ${PI/2}"/>
-        <geometry>
-          <cylinder length="${wheel_len}" radius="${wheel_radius}"/>
-        </geometry>
-        <material name="black"/>
-      </visual>
-      <inertial>
-        <origin xyz="0 0 0" rpy="${PI/2} 0 ${PI/2}"/>
-        <mass value="${wheel_mass}"/>
-        <inertia
-          ixx="0.000270" ixy="0.0" ixz="0.0"
-          iyy="0.000270" iyz="0.0"
-          izz="0.000426"/>
-      </inertial>
-    </link>
-    <joint name="${prefix}front_right_wheel_joint" type="revolute">
-      <parent link="${prefix}chassis_link" />
-      <child link="${prefix}front_right_wheel" />
-      <origin xyz="${wheelbase/2} ${base_width/2} -${base_height/2}" rpy="0 0 ${PI/2}"/>
-      <axis xyz="0 0 1"/>
-      <limit lower="-0.4" upper="0.4" effort="100.0" velocity="0.0"/>
-      <dynamics damping="0.2"/>
+      <inertial>
+        <origin xyz="0 0 0" rpy="${PI/2} 0 ${PI/2}"/>
+        <mass value="${wheel_mass}"/>
+        <inertia
+          ixx="0.001" ixy="0.0" ixz="0.0"
+          iyy="0.001" iyz="0.0"
+          izz="0.001"/>
+      </inertial>
+    </link>
+    <joint name="${prefix}front_right_wheel_joint" type="continuous">
+      <parent link="${prefix}chassis_link"/>
+      <child link="${prefix}front_right_wheel"/>
+      <origin xyz="${wheelbase} ${base_width/2} ${wheel_radius}" rpy="0 0 ${PI/2}"/>
+      <axis xyz="1 0 0"/>
+      <limit effort="10.0" velocity="10.0"/>
       <mimic joint="${prefix}virtual_front_wheel_joint" multiplier="1.0" offset="0.0"/>
     </joint>
-    <!-- front left steering -->
+    <!-- Front Left Wheel -->
     <link name="${prefix}front_left_wheel">
-      <collision>
-        <origin xyz="0 0 0" rpy="${PI/2} 0 ${PI/2}"/>
-        <geometry>
-          <cylinder length="${wheel_len}" radius="${wheel_radius}"/>
-        </geometry>
-      </collision>
-      <visual>
-        <origin xyz="0 0 0" rpy="${PI/2} 0 ${PI/2}"/>
-        <geometry>
-          <cylinder length="${wheel_len}" radius="${wheel_radius}"/>
-        </geometry>
-        <material name="black"/>
-      </visual>
-      <inertial>
-        <origin xyz="0 0 0" rpy="${PI/2} 0 ${PI/2}"/>
-        <mass value="${wheel_mass}"/>
-        <inertia
-          ixx="0.000270" ixy="0.0" ixz="0.0"
-          iyy="0.000270" iyz="0.0"
-          izz="0.000426"/>
-      </inertial>
-    </link>
-    <joint name="${prefix}front_left_wheel_joint" type="revolute">
-      <parent link="${prefix}chassis_link" />
-      <child link="${prefix}front_left_wheel" />
-      <origin xyz="${wheelbase/2} -${base_width/2} -${base_height/2}" rpy="0 0 ${PI/2}"/>
-      <axis xyz="0 0 1"/>
-      <limit lower="-0.4" upper="0.4" effort="100.0" velocity="0.0"/>
-      <dynamics damping="0.2"/>
+      <inertial>
+        <origin xyz="0 0 0" rpy="${PI/2} 0 ${PI/2}"/>
+        <mass value="${wheel_mass}"/>
+        <inertia
+          ixx="0.001" ixy="0.0" ixz="0.0"
+          iyy="0.001" iyz="0.0"
+          izz="0.001"/>
+      </inertial>
+    </link>
+    <joint name="${prefix}front_left_wheel_joint" type="continuous">
+      <parent link="${prefix}chassis_link"/>
+      <child link="${prefix}front_left_wheel"/>
+      <origin xyz="${wheelbase} -${base_width/2} ${wheel_radius}" rpy="0 0 ${PI/2}"/>
+      <axis xyz="1 0 0"/>
+      <limit effort="10.0" velocity="10.0"/>
       <mimic joint="${prefix}virtual_front_wheel_joint" multiplier="1.0" offset="0.0"/>
+    </joint>
+    <!-- LiDAR -->
+    <link name="${prefix}lidar_link">
+      <inertial>
+        <origin xyz="-0.036024 0 0.077736" rpy="0 0 0"/>
+        <mass value="0.2"/>
+        <inertia
+          ixx="0.0001" ixy="0.0" ixz="0.0"
+          iyy="0.0001" iyz="0.0"
+          izz="0.0001"/>
+      </inertial>
+    </link>
+    <joint name="${prefix}lidar_joint" type="fixed">
+      <parent link="${prefix}base_link"/>
+      <child link="${prefix}lidar_link"/>
+      <origin xyz="-0.036024 0 0.077736" rpy="0 0 0"/>
+    </joint>
+    <!-- IMU -->
+    <link name="${prefix}imu_link">
+      <inertial>
+        <origin xyz="0.1 0 0.01" rpy="0 0 0"/>
+        <mass value="0.1"/>
+        <inertia
+          ixx="0.0001" ixy="0.0" ixz="0.0"
+          iyy="0.0001" iyz="0.0"
+          izz="0.0001"/>
+      </inertial>
+    </link>
+    <joint name="${prefix}imu_joint" type="fixed">
+      <parent link="${prefix}chassis_link"/>
+      <child link="${prefix}imu_link"/>
+      <origin xyz="0.1 0 ${base_height + 0.03}" rpy="0 0 0"/>
+    </joint>
+    <!-- Color Sensors -->
+    <!-- Front Color Sensor -->
+    <link name="${prefix}front_color_sensor">
+      <inertial>
+        <origin xyz="${wheelbase} 0 ${base_height}" rpy="0 0 0"/>
+        <mass value="0.05"/>
+        <inertia
+          ixx="0.00005" ixy="0.0" ixz="0.0"
+          iyy="0.00005" iyz="0.0"
+          izz="0.00005"/>
+      </inertial>
+    </link>
+    <joint name="${prefix}front_color_sensor_joint" type="fixed">
+      <parent link="${prefix}chassis_link"/>
+      <child link="${prefix}front_color_sensor"/>
+      <origin xyz="${wheelbase} 0 ${base_height}" rpy="0 0 0"/>
+    </joint>
+    <!-- Rear Color Sensor -->
+    <link name="${prefix}rear_color_sensor">
+      <inertial>
+        <origin xyz="0 0 ${base_height}" rpy="0 0 0"/>
+        <mass value="0.05"/>
+        <inertia
+          ixx="0.00005" ixy="0.0" ixz="0.0"
+          iyy="0.00005" iyz="0.0"
+          izz="0.00005"/>
+      </inertial>
+    </link>
+    <joint name="${prefix}rear_color_sensor_joint" type="fixed">
+      <parent link="${prefix}chassis_link"/>
+      <child link="${prefix}rear_color_sensor"/>
+      <origin xyz="0 0 ${base_height}" rpy="0 0 0"/>
     </joint>
   </xacro:macro>

Commit message: urdf with base link in the middle of bot

File: src/description/urdf/carlikebot_description.urdf.xacro (robot description, xacro)
@@ -1,4 +1,4 @@
 <?xml version="1.0"?>
-<robot xmlns:xacro="http://www.ros.org/wiki/xacro" >
+<robot xmlns:xacro="http://www.ros.org/wiki/xacro" name="carlike_robot">
   <!-- Macro definition for carlikebot -->
   <xacro:macro name="carlikebot" params="prefix">
@@ -13,12 +13,4 @@
     <xacro:property name="wheel_len" value="0.05" />
     <xacro:property name="wheel_radius" value="0.1" />
-    <!--Property	Value (m)	Description
-base_width	0.408	Track width (distance between wheels on the same axle).
-base_length	0.558	Total length of the robot base.
-wheelbase	0.558	Distance between the front and rear wheel axles.
-wheel_radius	0.1	Radius of each wheel (half the diameter).
-wheel_len	0.05	Width of the wheels.
-base_height	0.06	Height of the chassis.
-base_mass	Approximate weight of the chassis (adjust if known).-->
     <!-- Base Link -->
     <link name="${prefix}base_link" />
@@ -37,20 +29,18 @@
       <parent link="${prefix}base_link"/>
       <child link="${prefix}chassis_link"/>
-      <origin xyz="${wheelbase/2} 0 ${2*wheel_radius}" rpy="0 0 0"/>
+      <origin xyz="0 0 ${base_height/2}" rpy="0 0 0"/>
+    </joint>
+    <!-- Virtual Rear Wheel -->
+    <link name="${prefix}virtual_rear_wheel" />
+    <joint name="${prefix}virtual_rear_wheel_joint" type="continuous">
+      <parent link="${prefix}chassis_link"/>
+      <child link="${prefix}virtual_rear_wheel"/>
+      <origin xyz="-${wheelbase/2} 0 ${wheel_radius}" rpy="0 0 ${PI/2}"/>
+      <axis xyz="1 0 0"/>
     </joint>
     <!-- Rear Wheels -->
-    <!-- Virtual Rear Wheel -->
-    <link name="${prefix}virtual_rear_wheel" />
-    <joint name="${prefix}virtual_rear_wheel_joint" type="revolute">
-      <parent link="${prefix}chassis_link"/>
-      <child link="${prefix}virtual_rear_wheel"/>
-      <origin xyz="${wheelbase/2} 0 ${wheel_radius}" rpy="0 0 ${PI/2}"/>
-      <axis xyz="0 0 1"/>
-      <limit lower="-0.4" upper="0.4" effort="10.0" velocity="10.0"/>
-    </joint>
-    <!-- Rear Right Wheel -->
     <link name="${prefix}rear_right_wheel">
       <inertial>
-        <origin xyz="0 0 0" rpy="${PI/2} 0 ${PI/2}"/>
+        <origin xyz="0 0 0" rpy="0 0 0"/>
         <mass value="${wheel_mass}"/>
         <inertia
@@ -63,13 +53,11 @@
       <parent link="${prefix}chassis_link"/>
       <child link="${prefix}rear_right_wheel"/>
-      <origin xyz="0 ${base_width/2} ${wheel_radius}" rpy="0 0 ${PI/2}"/>
+      <origin xyz="-${wheelbase/2} ${base_width/2} ${wheel_radius}" rpy="0 0 ${PI/2}"/>
       <axis xyz="1 0 0"/>
-      <limit effort="10.0" velocity="10.0"/>
       <mimic joint="${prefix}virtual_rear_wheel_joint" multiplier="1.0" offset="0.0"/>
     </joint>
-    <!-- Rear Left Wheel -->
     <link name="${prefix}rear_left_wheel">
       <inertial>
-        <origin xyz="0 0 0" rpy="${PI/2} 0 ${PI/2}"/>
+        <origin xyz="0 0 0" rpy="0 0 0"/>
         <mass value="${wheel_mass}"/>
         <inertia
@@ -82,23 +70,20 @@
       <parent link="${prefix}chassis_link"/>
       <child link="${prefix}rear_left_wheel"/>
-      <origin xyz="0 -${base_width/2} ${wheel_radius}" rpy="0 0 ${PI/2}"/>
+      <origin xyz="-${wheelbase/2} -${base_width/2} ${wheel_radius}" rpy="0 0 ${PI/2}"/>
       <axis xyz="1 0 0"/>
-      <limit effort="10.0" velocity="10.0"/>
       <mimic joint="${prefix}virtual_rear_wheel_joint" multiplier="1.0" offset="0.0"/>
     </joint>
-    <!-- Front Wheels -->
     <!-- Virtual Front Wheel -->
     <link name="${prefix}virtual_front_wheel" />
-    <joint name="${prefix}virtual_front_wheel_joint" type="revolute">
+    <joint name="${prefix}virtual_front_wheel_joint" type="continuous">
       <parent link="${prefix}chassis_link"/>
       <child link="${prefix}virtual_front_wheel"/>
       <origin xyz="${wheelbase/2} 0 ${wheel_radius}" rpy="0 0 ${PI/2}"/>
-      <axis xyz="0 0 1"/>
-      <limit lower="-0.4" upper="0.4" effort="10.0" velocity="10.0"/>
+      <axis xyz="1 0 0"/>
     </joint>
-    <!-- Front Right Wheel -->
+    <!-- Front Wheels -->
     <link name="${prefix}front_right_wheel">
       <inertial>
-        <origin xyz="0 0 0" rpy="${PI/2} 0 ${PI/2}"/>
+        <origin xyz="0 0 0" rpy="0 0 0"/>
         <mass value="${wheel_mass}"/>
         <inertia
@@ -111,13 +96,11 @@
       <parent link="${prefix}chassis_link"/>
       <child link="${prefix}front_right_wheel"/>
-      <origin xyz="${wheelbase} ${base_width/2} ${wheel_radius}" rpy="0 0 ${PI/2}"/>
+      <origin xyz="${wheelbase/2} ${base_width/2} ${wheel_radius}" rpy="0 0 ${PI/2}"/>
       <axis xyz="1 0 0"/>
-      <limit effort="10.0" velocity="10.0"/>
       <mimic joint="${prefix}virtual_front_wheel_joint" multiplier="1.0" offset="0.0"/>
     </joint>
-    <!-- Front Left Wheel -->
     <link name="${prefix}front_left_wheel">
       <inertial>
-        <origin xyz="0 0 0" rpy="${PI/2} 0 ${PI/2}"/>
+        <origin xyz="0 0 0" rpy="0 0 0"/>
         <mass value="${wheel_mass}"/>
         <inertia
@@ -130,7 +113,6 @@
       <parent link="${prefix}chassis_link"/>
       <child link="${prefix}front_left_wheel"/>
-      <origin xyz="${wheelbase} -${base_width/2} ${wheel_radius}" rpy="0 0 ${PI/2}"/>
+      <origin xyz="${wheelbase/2} -${base_width/2} ${wheel_radius}" rpy="0 0 ${PI/2}"/>
       <axis xyz="1 0 0"/>
-      <limit effort="10.0" velocity="10.0"/>
       <mimic joint="${prefix}virtual_front_wheel_joint" multiplier="1.0" offset="0.0"/>
     </joint>
@@ -138,5 +120,5 @@
     <link name="${prefix}lidar_link">
       <inertial>
-        <origin xyz="-0.036024 0 0.077736" rpy="0 0 0"/>
+        <origin xyz="0 0 0" rpy="0 0 0"/>
         <mass value="0.2"/>
         <inertia
@@ -151,53 +133,4 @@
       <origin xyz="-0.036024 0 0.077736" rpy="0 0 0"/>
     </joint>
-    <!-- IMU -->
-    <link name="${prefix}imu_link">
-      <inertial>
-        <origin xyz="0.1 0 0.01" rpy="0 0 0"/>
-        <mass value="0.1"/>
-        <inertia
-          ixx="0.0001" ixy="0.0" ixz="0.0"
-          iyy="0.0001" iyz="0.0"
-          izz="0.0001"/>
-      </inertial>
-    </link>
-    <joint name="${prefix}imu_joint" type="fixed">
-      <parent link="${prefix}chassis_link"/>
-      <child link="${prefix}imu_link"/>
-      <origin xyz="0.1 0 ${base_height + 0.03}" rpy="0 0 0"/>
-    </joint>
-    <!-- Color Sensors -->
-    <!-- Front Color Sensor -->
-    <link name="${prefix}front_color_sensor">
-      <inertial>
-        <origin xyz="${wheelbase} 0 ${base_height}" rpy="0 0 0"/>
-        <mass value="0.05"/>
-        <inertia
-          ixx="0.00005" ixy="0.0" ixz="0.0"
-          iyy="0.00005" iyz="0.0"
-          izz="0.00005"/>
-      </inertial>
-    </link>
-    <joint name="${prefix}front_color_sensor_joint" type="fixed">
-      <parent link="${prefix}chassis_link"/>
-      <child link="${prefix}front_color_sensor"/>
-      <origin xyz="${wheelbase} 0 ${base_height}" rpy="0 0 0"/>
-    </joint>
-    <!-- Rear Color Sensor -->
-    <link name="${prefix}rear_color_sensor">
-      <inertial>
-        <origin xyz="0 0 ${base_height}" rpy="0 0 0"/>
-        <mass value="0.05"/>
-        <inertia
-          ixx="0.00005" ixy="0.0" ixz="0.0"
-          iyy="0.00005" iyz="0.0"
-          izz="0.00005"/>
-      </inertial>
-    </link>
-    <joint name="${prefix}rear_color_sensor_joint" type="fixed">
-      <parent link="${prefix}chassis_link"/>
-      <child link="${prefix}rear_color_sensor"/>
-      <origin xyz="0 0 ${base_height}" rpy="0 0 0"/>
-    </joint>
   </xacro:macro>
 </robot>
