Commit message: color sensor urdf

File: src/description/urdf/carlikebot_description.urdf.xacro (robot description, xacro)
@@ -133,4 +133,35 @@
       <origin xyz="-0.036024 0 0.077736" rpy="0 0 0"/>
     </joint>
+<!-- Color Sensors -->
+  <link name="${prefix}front_color_sensor">
+    <inertial>
+      <origin xyz="${wheelbase} 0 ${base_height}" rpy="0 0 0"/>
+      <mass value="0.05"/>
+      <inertia
+        ixx="0.00005" ixy="0.0" ixz="0.0"
+        iyy="0.00005" iyz="0.0"
+        izz="0.00005"/>
+    </inertial>
+  </link>
+  <joint name="${prefix}front_color_sensor_joint" type="fixed">
+    <parent link="${prefix}chassis_link"/>
+    <child link="${prefix}front_color_sensor"/>
+    <origin xyz="${wheelbase} 0 ${base_height}" rpy="0 0 0"/>
+  </joint>
+  <link name="${prefix}rear_color_sensor">
+    <inertial>
+      <origin xyz="0 0 ${base_height}" rpy="0 0 0"/>
+      <mass value="0.05"/>
+      <inertia
+        ixx="0.00005" ixy="0.0" ixz="0.0"
+        iyy="0.00005" iyz="0.0"
+        izz="0.00005"/>
+    </inertial>
+  </link>
+  <joint name="${prefix}rear_color_sensor_joint" type="fixed">
+    <parent link="${prefix}chassis_link"/>
+    <child link="${prefix}rear_color_sensor"/>
+    <origin xyz="0 0 ${base_height}" rpy="0 0 0"/>
+  </joint>
   </xacro:macro>
 </robot>
